Commit message: Fix controls plugin. The urdf didnt recognize the plugin so <gazebo> tag had to be added to fix it

File: eklavya5_description/robots/chasisss.urdf.xacro (robot description, xacro)
@@ -439,3 +439,55 @@
         <material>Gazebo/White</material>
     </gazebo>
+    <!--<transmission type="SimpleTransmission" name="FrontWheel">
+      <type>transmission_interface/SimpleTransmission</type>
+      <joint name="Steerring Wheel" />
+      <actuator name="Steering_wheel_joint_motor">
+        <hardwareInterface>EffortJointInterface</hardwareInterface>
+        <mechanicalReduction>1</mechanicalReduction>
+      </actuator>
+  </transmission>
+  <transmission type="SimpleTransmission" name="LeftWheel">
+      <type>transmission_interface/SimpleTransmission</type>
+      <joint name="LW-Chassis" />
+      <actuator name="Left_wheel_joint_motor">
+        <hardwareInterface>EffortJointInterface</hardwareInterface>
+        <mechanicalReduction>1</mechanicalReduction>
+      </actuator>
+  </transmission>
+  <transmission type="SimpleTransmission" name="RightWheel">
+      <type>transmission_interface/SimpleTransmission</type>
+      <joint name="RW-Chassis" />
+      <actuator name="Right_wheel_joint_motor">
+        <hardwareInterface>EffortJointInterface</hardwareInterface>
+        <mechanicalReduction>1</mechanicalReduction>
+      </actuator>
+  </transmission>-->
+    <!-- Controls plugin-->
+  <gazebo>
+    <plugin filename="libeklavya_gazebo_plugins.so" name="eklavya_diff_controller">
+-      <alwaysOn>true</alwaysOn>
+-      <updateRate>100.0</updateRate>
+-      <backLeftJoint>joint_back_left_wheel</backLeftJoint>
+-      <backRightJoint>joint_back_right_wheel</backRightJoint>
+-      <frontLeftJoint>joint_front_left_wheel</frontLeftJoint>
+-      <!--<frontRightJoint>joint_front_right_wheel</frontRightJoint>-->
+-      <wheelSeparation>0.5709</wheelSeparation>
+-      <wheelDiameter>0.3555</wheelDiameter>
+-      <torque>35</torque>
+-    </plugin>
+     <!--<plugin name="gazebo_ros_control" filename="libgazebo_ros_control.so" />-->
+  </gazebo>
+-  <!--
+-  <gazebo>
+-    <plugin filename="libgazebo_ros_p3d.so" name="eklavya_groundtruth_sim">
+-      <updateRate>100.0</updateRate>
+-      <topicName>ground_truth/odom</topicName>
+-      <gaussianNoise>0.001</gaussianNoise>
+-      <frameName>world</frameName>
+-      <alwaysOn>true</alwaysOn>
+-      <bodyName>base_footprint</bodyName>
+-      <xyzOffset>0 0 0</xyzOffset>
+-      <rpyOffset>0 0 0</rpyOffset>
+-    </plugin>
+   </gazebo>-->
 </robot>

Commit message: Sensors converted to xacro. This made the raw code of chasisss.urdf.xacro concise, readable and modular.

File: eklavya5_description/robots/chasisss.urdf.xacro (robot description, xacro)
@@ -3,11 +3,15 @@
   name="chasisss"
   xmlns:sensor="http://playerstage.sourceforge.net/gazebo/xmlschema/#sensor"
-xmlns:controller="http://playerstage.sourceforge.net/gazebo/xmlschema/#controller"
-xmlns:interface="http://playerstage.sourceforge.net/gazebo/xmlschema/#interface"
-xmlns:xacro="http://ros.org/wiki/xacro"
->
-<xacro:include filename="$(find eklavya5_description)/sensors/imu.urdf.xacro" />
-<xacro:include filename="$(find eklavya5_description)/sensors/gps.urdf.xacro" />
- <property name="M_PI" value="3.1415926535897931" />
+  xmlns:controller="http://playerstage.sourceforge.net/gazebo/xmlschema/#controller"
+  xmlns:interface="http://playerstage.sourceforge.net/gazebo/xmlschema/#interface"
+  xmlns:xacro="http://ros.org/wiki/xacro">
+  <!-- Included URDF/XACRO Files -->
+  <xacro:include filename="$(find eklavya5_description)/sensors/camera.urdf.xacro" />
+  <xacro:include filename="$(find eklavya5_description)/sensors/lidar.urdf.xacro" />
+  <xacro:include filename="$(find eklavya5_description)/sensors/imu.urdf.xacro" />
+  <xacro:include filename="$(find eklavya5_description)/sensors/gps.urdf.xacro" />
+  <!-- PROPERTY LIST -->
+  <property name="M_PI" value="3.1415926535897931" />
+  <!--PARTS-->
   <link
     name = "base_link">
@@ -292,202 +296,39 @@
       velocity="0" />
   </joint>
-  <joint name="camera_joint" type="fixed">
-    <axis xyz="0 1 0" />
-    <origin xyz="0.05 0 0.5" rpy="0 0 0"/>
-    <parent link="Steering"/>
-    <child link="camera_link"/>
-  </joint>
+  <!--SENSORS-->
   <!-- Camera -->
-  <link name="camera_link">
-    <collision>
-      <origin xyz="0 0 0" rpy="0 0 0"/>
-      <geometry>
-    <box size="0.05 0.05 0.05"/>
-      </geometry>
-    </collision>
-    <visual>
-      <origin xyz="0 0 0" rpy="0 0 0"/>
-      <geometry>
-<box size="0.05 0.05 0.05"/>
-      </geometry>
-      <material name="red"/>
-    </visual>
-    <inertial>
-      <mass value="1e-5" />
-      <origin xyz="0 0 0" rpy="0 0 0"/>
-      <inertia ixx="1e-6" ixy="0" ixz="0" iyy="1e-6" iyz="0" izz="1e-6" />
-    </inertial>
-  </link>
-  <gazebo reference="camera_link">
-    <sensor type="camera" name="camera1">
-      <update_rate>24.0</update_rate>
-      <camera name="head">
-        <horizontal_fov>1.23</horizontal_fov>
-        <image>
-          <width>640</width>
-          <height>480</height>
-          <format>R8G8B8</format>
-        </image>
-        <clip>
-          <near>0.02</near>
-          <far>300</far>
-        </clip>
-        <noise>
-          <type>gaussian</type>
-          <!-- Noise is sampled independently per pixel on each frame.
-               That pixel's noise value is added to each of its color
-               channels, which at that point lie in the range [0,1]. -->
-          <mean>0.0</mean>
-          <stddev>0.007</stddev>
-        </noise>
-      </camera>
-      <plugin name="camera_controller" filename="libgazebo_ros_camera.so">
-        <alwaysOn>true</alwaysOn>
-        <updateRate>0.0</updateRate>
-        <cameraName>eklavya</cameraName>
-        <imageTopicName>image_raw</imageTopicName>
-        <cameraInfoTopicName>camera_info</cameraInfoTopicName>
-        <frameName>camera_link</frameName>
-        <hackBaseline>0.07</hackBaseline>
-        <distortionK1>0.0</distortionK1>
-        <distortionK2>0.0</distortionK2>
-        <distortionK3>0.0</distortionK3>
-        <distortionT1>0.0</distortionT1>
-        <distortionT2>0.0</distortionT2>
-      </plugin>
-    </sensor>
+  <sensor_camera parent="Steering" child="camera_link" name="camera" colour="Blue" camera_px="0.05" camera_py="0.0" camera_pz="0.5" camera_or="0.0" camera_op="0.0" camera_oy="0.0" axis_x="0" axis_y="1" axis_z="0"/>
+  <!-- Hokuyo Laser-->
+  <sensor_lidar parent="base_link" child="hokuyo_link" name="hokuyo" colour="Blue" lidar_px="-0.2" lidar_py="0.0" lidar_pz="0.8" lidar_or="0.0" lidar_op="0.0" lidar_oy="0.0" axis_x="0" axis_y="1" axis_z="0"/>
+  <!-- IMU-->
+  <sensor_imu parent="base_link" name="imu" colour="Blue" imu_px="-1" imu_py="0.0" imu_pz="0.8" imu_or="0.0" imu_op="${-M_PI/2.0}" imu_oy="0.0" />
+  <gazebo reference="imu_link">
+    <material>Gazebo/Blue</material>
   </gazebo>
-<!-- Hokuyo Laser-->
-<joint name="hokuyo_joint" type="fixed">
-    <axis xyz="0 1 0" />
-    <origin xyz="-0.2 0 0.8" rpy="0 0 0"/>
-    <parent link="base_link"/>
-    <child link="hokuyo_link"/>
-  </joint>
-  <link name="hokuyo_link">
-    <collision>
-      <origin xyz="0 0 0" rpy="0 0 0"/>
-      <geometry>
-    <box size="0.025 0.025 0.025"/>
-      </geometry>
-    </collision>
-    <visual>
-      <origin xyz="0 0 0" rpy="0 0 0"/>
-      <geometry>
-        <mesh filename="package://eklavya5_description/meshes/hokuyo.dae"/>
-      </geometry>
-    </visual>
-    <inertial>
-      <mass value="1e-5" />
-      <origin xyz="0 0 0" rpy="0 0 0"/>
-      <inertia ixx="1e-6" ixy="0" ixz="0" iyy="1e-6" iyz="0" izz="1e-6" />
-    </inertial>
-  </link>
-  <!-- hokuyo -->
-  <gazebo reference="hokuyo_link">
-    <sensor type="ray" name="head_hokuyo_sensor">
-      <pose>0 0 0 0 0 0</pose>
-      <visualize>true</visualize>
-      <update_rate>40</update_rate>
-      <ray>
-        <scan>
-          <horizontal>
-            <samples>720</samples>
-            <resolution>1</resolution>
-            <min_angle>-1.570796</min_angle>
-            <max_angle>1.570796</max_angle>
-          </horizontal>
-        </scan>
-        <range>
-          <min>0.1</min>
-          <max>4.0</max>
-          <resolution>0.01</resolution>
-        </range>
-        <noise>
-          <type>gaussian</type>
-          <!-- Noise parameters based on published spec for Hokuyo laser
-               achieving "+-30mm" accuracy at range < 10m.  A mean of 0.0m and
-               stddev of 0.01m will put 99.7% of samples within 0.03m of the true
-               reading. -->
-          <mean>0.0</mean>
-          <stddev>0.01</stddev>
-        </noise>
-      </ray>
-      <plugin name="gazebo_ros_head_hokuyo_controller" filename="libgazebo_ros_laser.so">
-        <topicName>eklavya/laser/scan</topicName>
-        <frameName>hokuyo_link</frameName>
-      </plugin>
-    </sensor>
+  <!-- GPS antenna/module -->
+  <sensor_gps parent="base_link" name="gps"
+        colour="White"
+        gps_px="-0.8"
+        gps_py="0"
+        gps_pz="0.8"
+        gps_or="0.0"
+        gps_op="0.0"
+        gps_oy="${M_PI}"
+        dimX="0.16" dimY="0.16" dimZ="0.14"/>
+  <gazebo reference="gps_link">
+      <material>Gazebo/White</material>
   </gazebo>
-<!-- IMU-->
-    <sensor_imu parent="base_link" name="imu" colour="Blue" imu_px="-1" imu_py="0.0" imu_pz="0.8" imu_or="0.0" imu_op="${-M_PI/2.0}" imu_oy="0.0" />
-    <gazebo reference="imu_link">
-        <material>Gazebo/Blue</material>
-    </gazebo>
-    <!-- GPS antenna/module -->
-    <sensor_gps parent="base_link" name="gps"
-          colour="White"
-          gps_px="-0.8"
-          gps_py="0"
-          gps_pz="0.8"
-          gps_or="0.0"
-          gps_op="0.0"
-          gps_oy="${M_PI}"
-          dimX="0.16" dimY="0.16" dimZ="0.14"
-          />
-    <gazebo reference="gps_link">
-        <material>Gazebo/White</material>
-    </gazebo>
-    <!--<transmission type="SimpleTransmission" name="FrontWheel">
-      <type>transmission_interface/SimpleTransmission</type>
-      <joint name="Steerring Wheel" />
-      <actuator name="Steering_wheel_joint_motor">
-        <hardwareInterface>EffortJointInterface</hardwareInterface>
-        <mechanicalReduction>1</mechanicalReduction>
-      </actuator>
-  </transmission>
-  <transmission type="SimpleTransmission" name="LeftWheel">
-      <type>transmission_interface/SimpleTransmission</type>
-      <joint name="LW-Chassis" />
-      <actuator name="Left_wheel_joint_motor">
-        <hardwareInterface>EffortJointInterface</hardwareInterface>
-        <mechanicalReduction>1</mechanicalReduction>
-      </actuator>
-  </transmission>
-  <transmission type="SimpleTransmission" name="RightWheel">
-      <type>transmission_interface/SimpleTransmission</type>
-      <joint name="RW-Chassis" />
-      <actuator name="Right_wheel_joint_motor">
-        <hardwareInterface>EffortJointInterface</hardwareInterface>
-        <mechanicalReduction>1</mechanicalReduction>
-      </actuator>
-  </transmission>-->
-    <!-- Controls plugin-->
+  <!-- CONTROLS PLUGIN-->
   <gazebo>
     <plugin filename="libeklavya_gazebo_plugins.so" name="eklavya_diff_controller">
--      <alwaysOn>true</alwaysOn>
--      <updateRate>100.0</updateRate>
--      <backLeftJoint>joint_back_left_wheel</backLeftJoint>
--      <backRightJoint>joint_back_right_wheel</backRightJoint>
--      <frontLeftJoint>joint_front_left_wheel</frontLeftJoint>
--      <!--<frontRightJoint>joint_front_right_wheel</frontRightJoint>-->
--      <wheelSeparation>0.5709</wheelSeparation>
--      <wheelDiameter>0.3555</wheelDiameter>
--      <torque>35</torque>
--    </plugin>
-     <!--<plugin name="gazebo_ros_control" filename="libgazebo_ros_control.so" />-->
+      <alwaysOn>true</alwaysOn>
+      <updateRate>100.0</updateRate>
+      <backLeftJoint>joint_back_left_wheel</backLeftJoint>
+      <backRightJoint>joint_back_right_wheel</backRightJoint>
+      <frontLeftJoint>joint_front_left_wheel</frontLeftJoint>
+      <wheelSeparation>0.5709</wheelSeparation>
+      <wheelDiameter>0.3555</wheelDiameter>
+      <torque>35</torque>
+    </plugin>
   </gazebo>
--  <!--
--  <gazebo>
--    <plugin filename="libgazebo_ros_p3d.so" name="eklavya_groundtruth_sim">
--      <updateRate>100.0</updateRate>
--      <topicName>ground_truth/odom</topicName>
--      <gaussianNoise>0.001</gaussianNoise>
--      <frameName>world</frameName>
--      <alwaysOn>true</alwaysOn>
--      <bodyName>base_footprint</bodyName>
--      <xyzOffset>0 0 0</xyzOffset>
--      <rpyOffset>0 0 0</rpyOffset>
--    </plugin>
-   </gazebo>-->
 </robot>
